Commit message: Add side boxes

File: marimbabot_sim/urdf/marimba.urdf.xacro (robot description, xacro)
@@ -4,6 +4,12 @@
 <xacro:include filename="$(find marimbabot_sim)/urdf/materials.xacro" />
 <!-- URDF/Gazebo model of a marimba.
+Coordinate system:
+From the point of view of the marimbist:
+    x: points towards you
+    y: points towards the right
+    z: points towards the ceiling, according to right hand rule
 Changelog:
     2023.03.02 Named and correctly positioned bar frames
+               Added side boxes
     2023.01.26 Complete model v1
     2023.01.19 Row of keys working
@@ -60,4 +66,12 @@
 <xacro:property name="top_left_center_y" value="${float(body_top_pos.split()[1]) - body_top_length / 2}" />
 <xacro:property name="top_left_center_z" value="${float(body_top_pos.split()[2]) + body_top_height / 2 + bar_height / 2}" />
+<!-- Side boxes (left being the longer side) -->
+<xacro:property name="side_width" value="0.05" />
+<xacro:property name="side_length_left" value="0.61" />
+<xacro:property name="side_length_right" value="0.32" />
+<xacro:property name="side_height" value="0.1" />
+<xacro:property name="side_offset" value="0.058" />
+<xacro:property name="side_left_pos" value="${(top_left_center_x + bottom_left_center_x) / 2} ${top_left_center_y - side_offset} ${bottom_left_center_z}" />
+<xacro:property name="side_right_pos" value="${float(side_left_pos.split()[0])} ${float(side_left_pos.split()[1]) + n_bars_bottom * (bar_width + bar_gap) - 1.5 * bar_gap + side_offset} ${float(side_left_pos.split()[2])}" />
 <!-- The bar -->
 <xacro:macro name="bar" params="note parent id pos length" >
@@ -124,5 +138,5 @@
             <!-- don't add the robotNamespace here unless you really want it -->
             <!-- <robotNamespace>${name}/</robotNamespace> -->
-            <!-- <robotNamespace>/</robotNamespace> -->
+            <!-- <robotNamespace>/</robotNamespaside_left_posce> -->
             <robotParam>robot_description</robotParam>
             <robotSimType>gazebo_ros_control/DefaultRobotHWSim</robotSimType>
@@ -200,4 +214,74 @@
     </link>
     <xacro:tams_fixedjoint name="body_top/fixedjoint" parent="${name}" child="body_top" >
+        <origin xyz="0 0 0" rpy="0 0 0" />
+    </xacro:tams_fixedjoint>
+    <!-- Left side box -->
+    <gazebo reference="body_left">
+        <turnGravityOff>false</turnGravityOff>
+        <selfCollide>false</selfCollide>
+        <!-- TODO material -->
+        <!-- <material>chordophones/OakWood</material> -->
+        <mu1>50.0</mu1>
+        <mu2>50.0</mu2>
+        <kp>1000000.0</kp>
+        <kd>1.0</kd>
+    </gazebo>
+    <link name="body_left">
+        <inertial>
+            <mass value="7.5" />
+            <origin xyz="0 0 0" rpy="0 0 0" />
+            <inertia ixx="0.2" ixy="0" ixz="0" iyy="0.2" iyz="0" izz="0.05" />
+        </inertial>
+        <visual>
+            <origin xyz="${side_left_pos}" rpy="0 0 1.57" />
+            <geometry>
+                <!-- <mesh filename="package://chordophones/meshes/guzheng-body.stl"  scale="0.001 0.001 0.001" /> -->
+                <box size="${side_width} ${side_length_left} ${side_height}"/>
+            </geometry>
+            <material name="gray" />
+        </visual>
+        <collision>
+            <origin xyz="${side_left_pos}" rpy="0 0 1.57" />
+            <geometry>
+                <box size="${side_width} ${side_length_left} ${side_height}"/>
+            </geometry>
+        </collision>
+    </link>
+    <xacro:tams_fixedjoint name="body_left/fixedjoint" parent="${name}" child="body_left" >
+        <origin xyz="0 0 0" rpy="0 0 0" />
+    </xacro:tams_fixedjoint>
+    <!-- Right side box -->
+    <gazebo reference="body_right">
+        <turnGravityOff>false</turnGravityOff>
+        <selfCollide>false</selfCollide>
+        <!-- TODO material -->
+        <!-- <material>chordophones/OakWood</material> -->
+        <mu1>50.0</mu1>
+        <mu2>50.0</mu2>
+        <kp>1000000.0</kp>
+        <kd>1.0</kd>
+    </gazebo>
+    <link name="body_right">
+        <inertial>
+            <mass value="7.5" />
+            <origin xyz="0 0 0" rpy="0 0 0" />
+            <inertia ixx="0.2" ixy="0" ixz="0" iyy="0.2" iyz="0" izz="0.05" />
+        </inertial>
+        <visual>
+            <origin xyz="${side_right_pos}" rpy="0 0 1.57" />
+            <geometry>
+                <!-- <mesh filename="package://chordophones/meshes/guzheng-body.stl"  scale="0.001 0.001 0.001" /> -->
+                <box size="${side_width} ${side_length_right} ${side_height}"/>
+            </geometry>
+            <material name="gray" />
+        </visual>
+        <collision>
+            <origin xyz="${side_right_pos}" rpy="0 0 1.57" />
+            <geometry>
+                <box size="${side_width} ${side_length_right} ${side_height}"/>
+            </geometry>
+        </collision>
+    </link>
+    <xacro:tams_fixedjoint name="body_right/fixedjoint" parent="${name}" child="body_right" >
         <origin xyz="0 0 0" rpy="0 0 0" />
     </xacro:tams_fixedjoint>

Commit message: Adjust body positions

File: marimbabot_sim/urdf/marimba.urdf.xacro (robot description, xacro)
@@ -34,5 +34,5 @@
 <xacro:property name="body_bottom_rpy" value="0 0 0.18" />
 <xacro:property name="body_bottom_length" value="0.82" />
-<xacro:property name="body_bottom_width" value="0.12" />
+<xacro:property name="body_bottom_width" value="0.2" />
 <xacro:property name="body_bottom_height" value="0.03" />
 <xacro:property name="body_bottom_slope" value="-0.35" />
@@ -60,10 +60,10 @@
 <xacro:property name="bottom_left_center_x" value="${float(body_bottom_pos.split()[0]) + bottom_left_offset}" />
 <xacro:property name="bottom_left_center_y" value="${float(body_bottom_pos.split()[1]) - body_bottom_length / 2}" />
-<xacro:property name="bottom_left_center_z" value="${float(body_bottom_pos.split()[1]) + body_bottom_height / 2 + bar_height / 2}" />
+<xacro:property name="bottom_left_center_z" value="${float(body_bottom_pos.split()[1]) + body_bottom_height / 2 + bar_height}" />
 <!-- Top row of bars starting pos (center of leftmost bar) -->
 <xacro:property name="top_left_offset" value="-0.03" />
 <xacro:property name="top_left_center_x" value="${float(body_top_pos.split()[0]) + top_left_offset}" />
 <xacro:property name="top_left_center_y" value="${float(body_top_pos.split()[1]) - body_top_length / 2}" />
-<xacro:property name="top_left_center_z" value="${float(body_top_pos.split()[2]) + body_top_height / 2 + bar_height / 2}" />
+<xacro:property name="top_left_center_z" value="${float(body_top_pos.split()[2]) + body_top_height / 2 + bar_height}" />
 <!-- Side boxes (left being the longer side) -->
 <xacro:property name="side_width" value="0.05" />

Commit message: Break long line

File: marimbabot_sim/urdf/marimba.urdf.xacro (robot description, xacro)
@@ -72,6 +72,14 @@
 <xacro:property name="side_height" value="0.1" />
 <xacro:property name="side_offset" value="0.058" />
-<xacro:property name="side_left_pos" value="${(top_left_center_x + bottom_left_center_x) / 2} ${top_left_center_y - side_offset} ${bottom_left_center_z}" />
-<xacro:property name="side_right_pos" value="${float(side_left_pos.split()[0])} ${float(side_left_pos.split()[1]) + n_bars_bottom * (bar_width + bar_gap) - 1.5 * bar_gap + side_offset} ${float(side_left_pos.split()[2])}" />
+<xacro:property name="side_left_pos" value="
+    ${(top_left_center_x + bottom_left_center_x) / 2}
+    ${top_left_center_y - side_offset}
+    ${bottom_left_center_z}"
+/>
+<xacro:property name="side_right_pos" value="
+    ${float(side_left_pos.split()[0])}
+    ${float(side_left_pos.split()[1]) + n_bars_bottom * (bar_width + bar_gap) - 1.5 * bar_gap + side_offset}
+    ${float(side_left_pos.split()[2])}"
+/>
 <!-- The bar -->
 <xacro:macro name="bar" params="note parent id pos length" >

Commit message: Specify gap between top & bottom row

File: marimbabot_sim/urdf/marimba.urdf.xacro (robot description, xacro)
@@ -44,5 +44,5 @@
 <xacro:property name="body_top_bottom_disp_x" value="-0.18" />
 <xacro:property name="body_top_bottom_disp_y" value="-0.02" />
-<xacro:property name="body_top_bottom_disp_z" value="0.03" />
+<xacro:property name="body_top_bottom_disp_z" value="${0.0149 + bar_height}" />
 <!-- Body top pos & dimensions -->
 <xacro:property name="body_top_pos" value="

Commit message: Fix robot to world

File: marimbabot_sim/urdf/marimba.urdf.xacro (robot description, xacro)
@@ -343,3 +343,9 @@
 <!-- TODO instantiate in standalone files -->
 <xacro:marimba name="marimba" />
+<link name="world"/>
+<joint name="fixed" type="fixed">
+    <parent link="world"/>
+    <child link="marimba"/>
+    <origin xyz="0 0 0" rpy="0 0 0" />
+</joint>
 </robot>

Commit message: Resolve review comments

File: marimbabot_sim/urdf/marimba.urdf.xacro (robot description, xacro)
@@ -341,11 +341,4 @@
     <xacro:bar_in_row note="A#6" parent="body_top" id="19" left_x="${top_left_center_x}" left_y="${top_left_center_y}" left_z="${top_left_center_z}" length_diff="${body_top_length_diff}" bar_length_left="${bar_length_top_left}" n_bars="${n_bars_top}" slope="${body_top_slope}" mirror="-1" />
 </xacro:macro>
-<!-- TODO instantiate in standalone files -->
 <xacro:marimba name="marimba" />
-<link name="world"/>
-<joint name="fixed" type="fixed">
-    <parent link="world"/>
-    <child link="marimba"/>
-    <origin xyz="0 0 0" rpy="0 0 0" />
-</joint>
 </robot>

File: marimbabot_sim/urdf/materials.xacro (robot description, xacro)
@@ -37,7 +37,3 @@
     <color rgba="1.0 1.0 1.0 1.0"/>
   </material>
-<!--
-  <material name="koto_wood">
-    <texture filename="file://$(find chordophones)/Media/materials/textures/koto.jpg" />
-  </material> -->
 </robot>
