Commit message: Updated URDF model. It can be launched with gazebo.roslaunch marimbabot_description  double_flex_mallet_gazebo.launch

File: marimbabot_description/urdf/double_flex_mallet.urdf (robot description, URDF)
Before this commit: robot double_flex_mallet, 1 links, 0 joints
Links:
- link base_link: mass None -> 0.36; geometry collision mesh filename=package://marimbabot_description/mesh/double_flex_v2_collis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 scale=0.001 0.001 0.001; visual mesh filename=package://marimbabot_description/mesh/mallet_mount_double_f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 scale=0.001 0.001 0.001
