Commit message: Improved the urdf-model for the Flex Mallet

File: marimbabot_description/urdf/flex_mallet_holder.urdf (robot description, URDF)
Before this commit: robot double_flex_mallet, 4 links, 3 joints
Joints:
- joint group_1_2nd_link: origin xyz=0.0 0.0 0.365 -> xyz=0.0 0.0 0.0

Commit message: Modiefied flex mallet holder

File: marimbabot_description/urdf/flex_mallet_holder.urdf (robot description, URDF)
Before this commit: robot double_flex_mallet, 4 links, 3 joints
Joints:
- joint group_1_2nd_link: origin xyz=0.0 0.0 0.0 -> xyz=0.0 0.0 0.397
- joint group_1_connector_plate_link: origin xyz=0.0 0.0 0.0118 -> xyz=0.0 0.0 -0.0059

Commit message: changed naming mallet

File: marimbabot_description/urdf/flex_mallet_holder.urdf (robot description, URDF)
Before this commit: robot double_flex_mallet, 4 links, 3 joints
Links:
- removed link mallet_top
- added link mallet_head; collision sphere radius=0.0198
Joints:
- joint group_1_2nd_link: child mallet_top -> mallet_head

Commit message: Added basic switchable attachments for the ur5

File: marimbabot_description/urdf/flex_mallet_holder.urdf (robot description, URDF)
Before this commit: robot double_flex_mallet, 4 links, 3 joints
Links:
- removed link base_link
- removed link connector_plate
- added link mallet_base_link; collision box size=0.090 0.0322 0.090; visual mesh filename=package://marimbabot_description/mesh/flex_mallet_holder.stl scale=0.001 0.001 0.001
- added link mallet_connector_plate; collision box size=0.05 0.0335 0.0118
Joints:
- joint group_1_connector_plate_link: child base_link -> mallet_base_link; parent connector_plate -> mallet_connector_plate
- joint group_1_start_link: parent base_link -> mallet_base_link

File: marimbabot_description/urdf/marimbabot_ur5.urdf.xacro (robot description, xacro)
@@ -3,4 +3,10 @@
        name="marimbabot_ur5" >
   <xacro:arg name="include_mallet" default="true" />
+  <!-- Choose the mallet holding assembly -->
+  <!-- Use 'static' for one mallet static holder -->
+  <!-- Use 'flex' for a flexible one mallet holder -->
+  <!-- Use 'flex_double' for the movable two mallet assembly with the flex holders -->
+  <xacro:arg name="mallet_holder_type" default="static" />
+  <xacro:property name="mallet_holder_type_param" value="$(arg mallet_holder_type)" />
   <!-- tams corner -->
   <xacro:include filename="$(find tams_ur5_setup_description)/urdf/tams_corner.urdf.xacro">
@@ -105,10 +111,28 @@
   </joint>
   <xacro:if value="$(arg include_mallet)">
-    <xacro:include filename="$(find marimbabot_description)/urdf/static_mallet_holder.urdf" />
-    <joint name="end_mallet" type="fixed">
-      <parent link="s_model_palm" />
-      <child link = "mallet_base_link" />
-      <origin xyz="0.0 0.0 0.0" rpy="${-pi/2} 0.0 0.0" />
-    </joint>
+    <xacro:if value="${mallet_holder_type_param == 'static'}">
+      <xacro:include filename="$(find marimbabot_description)/urdf/static_mallet_holder.urdf" />
+      <joint name="end_mallet" type="fixed">
+        <parent link="s_model_palm" />
+        <child link = "mallet_base_link" />
+        <origin xyz="0.0 0.0 0.0" rpy="${-pi/2} 0.0 0.0" />
+      </joint>
+    </xacro:if>
+    <xacro:if value="${mallet_holder_type_param == 'flex'}">
+      <xacro:include filename="$(find marimbabot_description)/urdf/flex_mallet_holder.urdf" />
+      <joint name="end_mallet" type="fixed">
+        <parent link="s_model_palm" />
+        <child link = "mallet_connector_plate" />
+        <origin xyz="0.0 ${(90/2+12)/1000} 0.0" rpy="${-pi/2} ${pi/2} 0.0" />
+      </joint>
+    </xacro:if>
+    <xacro:if value="${mallet_holder_type_param == 'double_flex'}">
+      <xacro:include filename="$(find marimbabot_description)/urdf/two_mallet_compliance_holder.urdf.xacro" />
+      <joint name="end_mallet" type="fixed">
+        <parent link="s_model_palm" />
+        <child link = "mallet_base_link" />
+        <origin xyz="0.0 0.0 0.0" rpy="${-pi/2} 0.0 0.0" />
+      </joint>
+    </xacro:if>
   </xacro:if>
 </robot>
