Commit message: add mallet configs

File: marimbabot_description/urdf/static_mallet_holder.urdf (robot description, URDF)
Before this commit: robot static_mallet_holder, 3 links, 2 joints
Links:
- removed link mallet_top
- added link mallet_head; collision sphere radius=0.018375
Joints:
- joint group_1_2nd_link: child mallet_top -> mallet_head

Commit message: Fixed static mallet holder mallet_head name and moved frame to center of sphere

File: marimbabot_description/urdf/static_mallet_holder.urdf (robot description, URDF)
Before this commit: robot static_mallet_holder, 3 links, 2 joints
Links:
- removed link mallet_top
- added link mallet_head, mass 0.01; collision sphere radius=0.018375; visual sphere radius=0.018375
Joints:
- joint group_1_2nd_link: origin xyz=0.0 0.0 0.365 -> xyz=0.0 0.0 0.378625

Commit message: adjust mallet length based on real time experiments

File: marimbabot_description/urdf/static_mallet_holder.urdf (robot description, URDF)
Before this commit: robot static_mallet_holder, 3 links, 2 joints
Joints:
- joint group_1_2nd_link: origin xyz=0.0 0.0 0.378625 -> xyz=0.0 0.0 0.468625
