Commit message: add mallet to the model

File: marimbabot_description/urdf/marimbabot_ur5.urdf.xacro (robot description, xacro)
@@ -10,4 +10,5 @@
   <xacro:include filename="$(find tams_ur5_description)/urdf/arm.urdf.xacro" />
   <xacro:include filename="$(find marimbabot_description)/urdf/marimba.urdf.xacro" />
+  <xacro:include filename="$(find marimbabot_description)/urdf/static_mallet_holder.urdf" />
   <link name="world" />
   <joint name="world_floor_joint" type="fixed">
@@ -32,3 +33,8 @@
     <origin xyz="0.9 0.8 0.9" rpy="0.0 0.0 ${pi}" />
   </joint>
+  <joint name="end_mallet" type="fixed">
+    <parent link="s_model_palm" />
+    <child link = "mallet_base_link" />
+    <origin xyz="0.0 0.0 0.0" rpy="${-pi/2} 0.0 0.0" />
+  </joint>
 </robot>

File: marimbabot_description/urdf/static_mallet_holder.urdf (robot description, URDF)
Before this commit: robot static_mallet_holder, 3 links, 2 joints
Links:
- removed link base_link
- added link mallet_base_link; collision box size=0.024 0.024 0.0992; visual mesh filename=package://marimbabot_description/mesh/static_mallet_holder.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 scale=0.001 0.001 0.001
Joints:
- joint group_1_start_link: parent base_link -> mallet_base_link

Commit message: WIP gazebo

File: marimbabot_description/urdf/marimbabot_ur5.urdf.xacro (robot description, xacro)
@@ -2,4 +2,6 @@
 <robot xmlns:xacro="http://www.ros.org/wiki/xacro"
        name="marimbabot_ur5" >
+  <xacro:arg name="r200" default="false" />
+  <xacro:arg name="include_mallet" default="true" />
   <!-- tams corner -->
   <xacro:include filename="$(find tams_ur5_setup_description)/urdf/tams_corner.urdf.xacro">
@@ -7,9 +9,97 @@
   <!-- the above argument is ignored by xacro! if you want to use this argument, try another way -->
   </xacro:include>
-  <!-- arm -->
-  <xacro:include filename="$(find tams_ur5_description)/urdf/arm.urdf.xacro" />
+  <!-- fnh: was <xacro:include filename="$(find tams_ur5_description)/urdf/arm.urdf.xacro" /> -->
+  <!-- arm plus additions one by one -->  <!-- include macro definitions -->
+  <xacro:include filename="$(find tams_ur5_gazebo)/urdf/ur5_for_gazebo.urdf.xacro" />
+  <xacro:include filename="$(find robotiq_3f_gripper_visualization)/cfg/robotiq-3f-gripper_articulated_macro.xacro"/>
+  <xacro:include filename="$(find robotiq_ft_sensor)/urdf/robotiq_fts150.urdf.xacro" />
+  <xacro:include filename="$(find tams_ur5_description)/urdf/ft_adapter.urdf.xacro" />
+  <xacro:include filename="$(find tams_ur5_description)/urdf/s_model_adapter.urdf.xacro" />
+  <xacro:include filename="$(find tams_ur5_description)/urdf/plug_collision_model.urdf.xacro" />
   <xacro:include filename="$(find marimbabot_description)/urdf/marimba.urdf.xacro" />
-  <xacro:include filename="$(find marimbabot_description)/urdf/gazebo_gripper_transmissions.xacro" />
-  <xacro:include filename="$(find marimbabot_description)/urdf/static_mallet_holder.urdf" />
+  <!-- <xacro:include filename="$(find marimbabot_description)/urdf/gazebo_gripper_transmissions.xacro" /> -->
+  <xacro:if value="$(arg include_mallet)">
+    <xacro:include filename="$(find marimbabot_description)/urdf/static_mallet_holder.urdf" />
+  </xacro:if>
+  <!-- fnh: arm with xamla_cap and gazebo EffortJointInterface transmissions -->
+  <!-- fnh: uncommented universal_robot/ur_description/urdf/common.gazebo.xacro -->
+  <!-- fnh: also removed the hardcoded PositionJointInterface transmissions. See below for hotfix -->
+  <xacro:ur5_robot prefix="ur5_" joint_limited="false" xamla_cap="true" />
+  <!-- ft_adapter -->
+  <xacro:ft_adapter name="ft_adapter" parent="ur5_ee_link">
+    <origin xyz="0.0045 0.0 0.0" rpy="0.0 ${pi/2} 0.0" />
+  </xacro:ft_adapter>
+  <!-- mounted_camera -->
+  <xacro:if value="$(arg r200)">
+    <xacro:mounted_camera name="mounted_camera" parent="ft_adapter">
+        <origin xyz="0 0 0.0" rpy="0 0 0" />
+    </xacro:mounted_camera>
+    <!-- gazebo camera plugin should go here -->
+  </xacro:if>
+  <!-- ft150 -->
+  <xacro:robotiq_fts150 prefix="ft_" parent="ur5_ee_link">
+    <origin xyz="0.009 0.0 0.0" rpy="0.0 ${-pi/2} ${pi}" />
+  </xacro:robotiq_fts150>
+  <!-- tool0 frame -->
+  <link name="tool0" />
+  <joint name="ft_fts_toolside_tool0" type="fixed">
+    <parent link="ft_fts_toolside"/>
+    <child link="tool0"/>
+    <origin xyz="0.0 0.0 0.0205" rpy="0.0 ${-pi/2} 0.0"/>
+  </joint>
+  <!-- s_model_adapter -->
+  <xacro:s_model_adapter name="s_model_adapter" parent="ft_fts_toolside">
+    <origin xyz="0.0 0.0 0.015" rpy="0.0 0.0 0.0" />
+  </xacro:s_model_adapter>
+  <!-- the adaptive gripper -->
+  <xacro:robotiq-3f-gripper_articulated prefix="s_model_"/>
+  <joint name="gripper_joint" type="fixed">
+    <parent link="tool0" />
+    <child link = "s_model_palm" />
+    <origin xyz="0.057 0.0 0.0" rpy="0.0 ${pi} ${-pi/2}" />
+  </joint>
+  <!-- plug collision model -->
+  <xacro:plug_collision_model name="plug_collision_model" parent="ur5_ee_link" >
+    <origin xyz="0.0 0.0 0.0" rpy="0.0 0.0 0.0" />
+  </xacro:plug_collision_model>
+  <!-- we want Gazebo to publish joint_states for all configured joints -->
+  <gazebo>
+    <plugin filename="libgazebo_ros_control.so" name="tams_ur5_gazebo_ros_control">
+      <!-- <robotSimType>sr_gazebo_sim/SrGazeboHWSim</robotSimType> -->
+      <robotNamespace>/</robotNamespace>
+      <robotSimType>gazebo_ros_control/DefaultRobotHWSim</robotSimType>
+      <legacyModeNS>true</legacyModeNS>
+      <updateRate>100.0</updateRate>
+    </plugin>
+  </gazebo>
+  <!-- fnh: some EffortJointInterface transmissions, UR and Robotiq repos do not have them  -->
+  <xacro:macro name="fake_transmission" params="joint_name" >
+    <transmission name="${joint_name}_transmission">
+      <type>transmission_interface/SimpleTransmission</type>
+      <actuator name="${joint_name}_motor">
+        <mechanicalReduction>1.0</mechanicalReduction>
+      </actuator>
+      <joint name="${joint_name}">
+        <hardwareInterface>hardware_interface/EffortJointInterface</hardwareInterface>
+      </joint>
+    </transmission>
+  </xacro:macro>
+  <xacro:fake_transmission joint_name="ur5_shoulder_pan_joint" />
+  <xacro:fake_transmission joint_name="ur5_shoulder_lift_joint" />
+  <xacro:fake_transmission joint_name="ur5_elbow_joint" />
+  <xacro:fake_transmission joint_name="ur5_wrist_1_joint" />
+  <xacro:fake_transmission joint_name="ur5_wrist_2_joint" />
+  <xacro:fake_transmission joint_name="ur5_wrist_3_joint" />
+  <xacro:fake_transmission joint_name="s_model_palm_finger_1_joint" />
+  <xacro:fake_transmission joint_name="s_model_finger_1_joint_1" />
+  <xacro:fake_transmission joint_name="s_model_finger_1_joint_2" />
+  <xacro:fake_transmission joint_name="s_model_finger_1_joint_3" />
+  <xacro:fake_transmission joint_name="s_model_palm_finger_2_joint" />
+  <xacro:fake_transmission joint_name="s_model_finger_2_joint_1" />
+  <xacro:fake_transmission joint_name="s_model_finger_2_joint_2" />
+  <xacro:fake_transmission joint_name="s_model_finger_2_joint_3" />
+  <xacro:fake_transmission joint_name="s_model_finger_middle_joint_1" />
+  <xacro:fake_transmission joint_name="s_model_finger_middle_joint_2" />
+  <xacro:fake_transmission joint_name="s_model_finger_middle_joint_3" />
   <link name="world" />
   <joint name="world_floor_joint" type="fixed">

File: marimbabot_description/urdf/static_mallet_holder.urdf (robot description, URDF)
Before this commit: robot static_mallet_holder, 3 links, 2 joints
Links:
- link mallet_base_link: mass None -> 0.005
- link mallet_neck: mass None -> 0.001; geometry collision cylinder length=0.375 radius=0.0042; visual cylinder length=0.375 radius=0.0042
- link mallet_top: mass None -> 0.01; geometry collision sphere radius=0.018375; visual sphere radius=0.018375

Commit message: conditional loading for mallet

File: marimbabot_description/urdf/marimbabot_ur5.urdf.xacro (robot description, xacro)
@@ -19,7 +19,4 @@
   <xacro:include filename="$(find marimbabot_description)/urdf/marimba.urdf.xacro" />
   <!-- <xacro:include filename="$(find marimbabot_description)/urdf/gazebo_gripper_transmissions.xacro" /> -->
-  <xacro:if value="$(arg include_mallet)">
-    <xacro:include filename="$(find marimbabot_description)/urdf/static_mallet_holder.urdf" />
-  </xacro:if>
   <!-- fnh: arm with xamla_cap and gazebo EffortJointInterface transmissions -->
   <!-- fnh: uncommented universal_robot/ur_description/urdf/common.gazebo.xacro -->
@@ -124,8 +121,11 @@
     <origin xyz="0.9 0.8 0.9" rpy="0.0 0.0 ${pi}" />
   </joint>
-  <joint name="end_mallet" type="fixed">
-    <parent link="s_model_palm" />
-    <child link = "mallet_base_link" />
-    <origin xyz="0.0 0.0 0.0" rpy="${-pi/2} 0.0 0.0" />
-  </joint>
+  <xacro:if value="$(arg include_mallet)">
+    <xacro:include filename="$(find marimbabot_description)/urdf/static_mallet_holder.urdf" />
+    <joint name="end_mallet" type="fixed">
+      <parent link="s_model_palm" />
+      <child link = "mallet_base_link" />
+      <origin xyz="0.0 0.0 0.0" rpy="${-pi/2} 0.0 0.0" />
+    </joint>
+  </xacro:if>
 </robot>

Commit message: Move marimba further away

File: marimbabot_description/urdf/marimbabot_ur5.urdf.xacro (robot description, xacro)
@@ -31,5 +31,5 @@
     <parent link="world" />
     <child link = "marimba" />
-    <origin xyz="0.9 0.8 0.9" rpy="0.0 0.0 ${pi}" />
+    <origin xyz="1.25 0.8 0.9" rpy="0.0 0.0 ${pi}" />
   </joint>
   <joint name="end_mallet" type="fixed">

Commit message: remove comments

File: marimbabot_description/urdf/marimbabot_ur5.urdf.xacro (robot description, xacro)
@@ -2,12 +2,8 @@
 <robot xmlns:xacro="http://www.ros.org/wiki/xacro"
        name="marimbabot_ur5" >
-  <xacro:arg name="r200" default="false" />
   <xacro:arg name="include_mallet" default="true" />
   <!-- tams corner -->
   <xacro:include filename="$(find tams_ur5_setup_description)/urdf/tams_corner.urdf.xacro">
-  <!-- <xacro:arg name="floating_table" value="$(arg floating_table)" />-->
-  <!-- the above argument is ignored by xacro! if you want to use this argument, try another way -->
   </xacro:include>
-  <!-- fnh: was <xacro:include filename="$(find tams_ur5_description)/urdf/arm.urdf.xacro" /> -->
   <!-- arm plus additions one by one -->  <!-- include macro definitions -->
   <xacro:include filename="$(find tams_ur5_gazebo)/urdf/ur5_for_gazebo.urdf.xacro" />
@@ -18,8 +14,4 @@
   <xacro:include filename="$(find tams_ur5_description)/urdf/plug_collision_model.urdf.xacro" />
   <xacro:include filename="$(find marimbabot_description)/urdf/marimba.urdf.xacro" />
-  <!-- <xacro:include filename="$(find marimbabot_description)/urdf/gazebo_gripper_transmissions.xacro" /> -->
-  <!-- fnh: arm with xamla_cap and gazebo EffortJointInterface transmissions -->
-  <!-- fnh: uncommented universal_robot/ur_description/urdf/common.gazebo.xacro -->
-  <!-- fnh: also removed the hardcoded PositionJointInterface transmissions. See below for hotfix -->
   <xacro:ur5_robot prefix="ur5_" joint_limited="false" xamla_cap="true" />
   <!-- ft_adapter -->
@@ -27,11 +19,4 @@
     <origin xyz="0.0045 0.0 0.0" rpy="0.0 ${pi/2} 0.0" />
   </xacro:ft_adapter>
-  <!-- mounted_camera -->
-  <xacro:if value="$(arg r200)">
-    <xacro:mounted_camera name="mounted_camera" parent="ft_adapter">
-        <origin xyz="0 0 0.0" rpy="0 0 0" />
-    </xacro:mounted_camera>
-    <!-- gazebo camera plugin should go here -->
-  </xacro:if>
   <!-- ft150 -->
   <xacro:robotiq_fts150 prefix="ft_" parent="ur5_ee_link">
@@ -63,5 +48,4 @@
   <gazebo>
     <plugin filename="libgazebo_ros_control.so" name="tams_ur5_gazebo_ros_control">
-      <!-- <robotSimType>sr_gazebo_sim/SrGazeboHWSim</robotSimType> -->
       <robotNamespace>/</robotNamespace>
       <robotSimType>gazebo_ros_control/DefaultRobotHWSim</robotSimType>
@@ -70,5 +54,4 @@
     </plugin>
   </gazebo>
-  <!-- fnh: some EffortJointInterface transmissions, UR and Robotiq repos do not have them  -->
   <xacro:macro name="fake_transmission" params="joint_name" >
     <transmission name="${joint_name}_transmission">

Commit message: Load marimba and arm setup separately in Gazebo

File: marimbabot_description/urdf/marimbabot_ur5.urdf.xacro (robot description, xacro)
@@ -13,5 +13,4 @@
   <xacro:include filename="$(find tams_ur5_description)/urdf/s_model_adapter.urdf.xacro" />
   <xacro:include filename="$(find tams_ur5_description)/urdf/plug_collision_model.urdf.xacro" />
-  <xacro:include filename="$(find marimbabot_description)/urdf/marimba.urdf.xacro" />
   <xacro:ur5_robot prefix="ur5_" joint_limited="false" xamla_cap="true" />
   <!-- ft_adapter -->
@@ -99,9 +98,9 @@
     <origin xyz="0 0 0.003" rpy="0.0 0.0 ${pi/2}" />
   </joint>
-  <joint name="world_marimba_joint" type="fixed">
+  <!-- <joint name="world_marimba_joint" type="fixed">
     <parent link="world" />
     <child link = "marimba" />
     <origin xyz="1.25 0.8 0.9" rpy="0.0 0.0 ${pi}" />
-  </joint>
+  </joint> -->
   <xacro:if value="$(arg include_mallet)">
     <xacro:include filename="$(find marimbabot_description)/urdf/static_mallet_holder.urdf" />

File: marimbabot_hardware/urdf/two_mallet_holder.urdf (robot description, URDF)
Before this commit: robot two_mallet_holder, 2 links, 1 joints
Links:
- removed link mallet_top
- added link mallet_head; collision sphere radius=0.018375

Commit message: Adjusted positioning of two mallet holder + extended readme

File: marimbabot_description/urdf/marimbabot_ur5.urdf.xacro (robot description, xacro)
@@ -132,5 +132,5 @@
         <parent link="s_model_palm" />
         <child link = "mallet_base_link" />
-        <origin xyz="0.0 0.0 0.0" rpy="${-pi/2} 0.0 0.0" />
+        <origin xyz="0.0 ${(80+11)/1000} ${(-45)/1000}" rpy="0.0 0.0 ${pi}" />
       </joint>
     </xacro:if>

Commit message: modify marimba height based on real experiments

File: marimbabot_description/urdf/marimbabot_ur5.urdf.xacro (robot description, xacro)
@@ -102,5 +102,5 @@
     <parent link="world" />
     <child link = "marimba" />
-    <origin xyz="1.25 0.8 0.9" rpy="0.0 0.0 ${pi}" />
+    <origin xyz="1.25 0.8 0.80" rpy="0.0 0.0 ${pi}" />
   </joint>
   <xacro:if value="$(arg include_mallet)">

Commit message: Adjusted the base link offset of the double mallet

File: marimbabot_description/urdf/marimbabot_ur5.urdf.xacro (robot description, xacro)
@@ -132,5 +132,5 @@
         <parent link="s_model_palm" />
         <child link = "mallet_base_link" />
-        <origin xyz="0.0 ${(80+11)/1000} ${(-45)/1000}" rpy="0.0 0.0 ${pi}" />
+        <origin xyz="0.0 ${(80+11)/1000} ${(-48)/1000}" rpy="0.0 0.0 ${pi}" />
       </joint>
     </xacro:if>

Commit message: Move marimba closer to the robot

File: marimbabot_description/urdf/marimbabot_ur5.urdf.xacro (robot description, xacro)
@@ -108,5 +108,5 @@
     <parent link="world" />
     <child link = "marimba" />
-    <origin xyz="1.25 0.8 0.80" rpy="0.0 0.0 ${pi}" />
+    <origin xyz="1.0 0.8 0.80" rpy="0.0 0.0 ${pi}" />
   </joint>
   <xacro:if value="$(arg include_mallet)">
