Commit message: Move sim package to description

File: marimbabot_description/urdf/marimba.urdf.xacro (robot description, xacro)
@@ -1,6 +1,6 @@
 <?xml version="1.0" ?>
 <robot name="marimba" xmlns:xacro="http://www.ros.org/wiki/xacro">
-<xacro:include filename="$(find marimbabot_sim)/urdf/utilities.xacro" />
-<xacro:include filename="$(find marimbabot_sim)/urdf/materials.xacro" />
+<xacro:include filename="$(find marimbabot_description)/urdf/utilities.xacro" />
+<xacro:include filename="$(find marimbabot_description)/urdf/materials.xacro" />
 <!-- URDF/Gazebo model of a marimba.
 Coordinate system:

File: marimbabot_description/urdf/materials.xacro (robot description, xacro)
@@ -1,26 +1,26 @@
 <?xml version="1.0"?>
 <robot xmlns:xacro="http://www.ros.org/wiki/xacro">
-  <material name="black">
+  <!-- <material name="black">
     <color rgba="0.0 0.0 0.0 1.0"/>
-  </material>
-  <material name="blue">
+  </material> -->
+  <!-- <material name="blue">
     <color rgba="0.0 0.0 0.8 1.0"/>
   </material>
   <material name="green">
     <color rgba="0.0 0.8 0.0 1.0"/>
-  </material>
+  </material> -->
   <material name="gray">
     <color rgba="0.2 0.2 0.2 1.0"/>
   </material>
-  <material name="lightgray">
+  <!-- <material name="lightgray">
     <color rgba="0.6 0.6 0.6 1.0"/>
   </material>
   <material name="darkgray">
     <color rgba="0.4 0.4 0.4 1.0"/>
-  </material>
+  </material> -->
   <material name="red">
     <color rgba="0.9 0.0 0.0 1.0"/>
   </material>
-  <material name="orange">
+  <!-- <material name="orange">
     <color rgba="0.95 0.64 0.0 1.0"/>
   </material>
@@ -36,4 +36,4 @@
   <material name="white">
     <color rgba="1.0 1.0 1.0 1.0"/>
-  </material>
+  </material> -->
 </robot>

Commit message: Fix color and collision boxes

File: marimbabot_description/urdf/marimba.urdf.xacro (robot description, xacro)
@@ -76,5 +76,5 @@
     ${top_left_center_y - side_offset}
     ${bottom_left_center_z}"
-/>
+/>re
 <xacro:property name="side_right_pos" value="
     ${float(side_left_pos.split()[0])}
@@ -103,12 +103,11 @@
         <!-- TODO material -->
         <!-- <material name="oak_wood" /> -->
-        <material name="red" />
+        <material name="marimba_key" />
     </visual>
     <collision>
-        <origin xyz="0 0 0" rpy="0 0 0" />
+        <origin xyz="0 0 ${-bar_height / 2}" rpy="0 0 0" />
         <geometry>
-            <box size="${bar_width} ${bar_height} ${length}"/>
+            <box size="${length} ${bar_width} ${bar_height}"/>
         </geometry>
-        <material name="blue" />
     </collision>
     </link>

File: marimbabot_description/urdf/materials.xacro (robot description, xacro)
@@ -19,6 +19,6 @@
     <color rgba="0.4 0.4 0.4 1.0"/>
   </material> -->
-  <material name="red">
-    <color rgba="0.9 0.0 0.0 1.0"/>
+  <material name="marimba_key">
+    <color rgba="0.5 0.3 0.1 1.0"/>
   </material>
   <!-- <material name="orange">

Commit message: WIP: Gazebo simulation

File: marimbabot_description/urdf/marimba.urdf.xacro (robot description, xacro)
@@ -10,4 +10,5 @@
     z: points towards the ceiling, according to right hand rule
 Changelog:
+    2023.04.20 TODO
     2023.03.02 Named and correctly positioned bar frames
                Added side boxes
@@ -15,6 +16,4 @@
     2023.01.19 Row of keys working
     2023.01.04 First version created
-TODO:
-    - prismatic joints instead of fixed ones for the bars
 -->
 <!-- Number of bars (including "missing" ones in the top row) -->
@@ -112,7 +111,16 @@
     </collision>
     </link>
-    <xacro:tams_fixedjoint name="bar_${note}/fixedjoint" parent="${parent}" child="bar_${note}" >
+    <xacro:tams_z_joint name="bar_${note}/joint" parent="${parent}" child="bar_${note}" >
         <origin xyz="${pos}" rpy="0 0 0" />
-    </xacro:tams_fixedjoint>
+    </xacro:tams_z_joint>
+    <transmission name="bar_${note}/joint_transmission">
+        <type>transmission_interface/SimpleTransmission</type>
+        <joint name="bar_${note}/joint">
+        <hardwareInterface>hardware_interface/EffortJointInterface</hardwareInterface>
+        </joint>
+        <actuator name="bar_${note}/joint_motor">
+        <mechanicalReduction>1</mechanicalReduction>
+        </actuator>
+    </transmission>
 </xacro:macro>
 <!-- Wrapper for a row of bars, computes the position and length based on fixed measurements -->
@@ -144,5 +152,5 @@
         <plugin filename="libgazebo_ros_control.so" name="${name}_gazebo_ros_control">
             <!-- don't add the robotNamespace here unless you really want it -->
-            <!-- <robotNamespace>${name}/</robotNamespace> -->
+            <!-- <robotNamespace>marimba/</robotNamespace> -->
             <!-- <robotNamespace>/</robotNamespaside_left_posce> -->
             <robotParam>robot_description</robotParam>
@@ -319,24 +327,24 @@
     <!-- Top row of bars -->
     <xacro:property name="body_top_length_diff" value="${bar_length_top_right - bar_length_top_left}" />
-    <xacro:bar_in_row note="C#4" parent="body_top" id="0" left_x="${top_left_center_x}" left_y="${top_left_center_y}" left_z="${top_left_center_z}" length_diff="${body_top_length_diff}" bar_length_left="${bar_length_top_left}" n_bars="${n_bars_top}" slope="${body_top_slope}" mirror="-1" />
-    <xacro:bar_in_row note="D#4" parent="body_top" id="1" left_x="${top_left_center_x}" left_y="${top_left_center_y}" left_z="${top_left_center_z}" length_diff="${body_top_length_diff}" bar_length_left="${bar_length_top_left}" n_bars="${n_bars_top}" slope="${body_top_slope}" mirror="-1" />
+    <xacro:bar_in_row note="Cs4" parent="body_top" id="0" left_x="${top_left_center_x}" left_y="${top_left_center_y}" left_z="${top_left_center_z}" length_diff="${body_top_length_diff}" bar_length_left="${bar_length_top_left}" n_bars="${n_bars_top}" slope="${body_top_slope}" mirror="-1" />
+    <xacro:bar_in_row note="Ds4" parent="body_top" id="1" left_x="${top_left_center_x}" left_y="${top_left_center_y}" left_z="${top_left_center_z}" length_diff="${body_top_length_diff}" bar_length_left="${bar_length_top_left}" n_bars="${n_bars_top}" slope="${body_top_slope}" mirror="-1" />
     <!-- <xacro:bar_in_row note="" parent="body_top" id="2" left_x="${top_left_center_x}" left_y="${top_left_center_y}" left_z="${top_left_center_z}" length_diff="${body_top_length_diff}" bar_length_left="${bar_length_top_left}" n_bars="${n_bars_top}" slope="${body_top_slope}" mirror="-1" /> -->
-    <xacro:bar_in_row note="F#4" parent="body_top" id="3" left_x="${top_left_center_x}" left_y="${top_left_center_y}" left_z="${top_left_center_z}" length_diff="${body_top_length_diff}" bar_length_left="${bar_length_top_left}" n_bars="${n_bars_top}" slope="${body_top_slope}" mirror="-1" />
-    <xacro:bar_in_row note="G#4" parent="body_top" id="4" left_x="${top_left_center_x}" left_y="${top_left_center_y}" left_z="${top_left_center_z}" length_diff="${body_top_length_diff}" bar_length_left="${bar_length_top_left}" n_bars="${n_bars_top}" slope="${body_top_slope}" mirror="-1" />
-    <xacro:bar_in_row note="A#4" parent="body_top" id="5" left_x="${top_left_center_x}" left_y="${top_left_center_y}" left_z="${top_left_center_z}" length_diff="${body_top_length_diff}" bar_length_left="${bar_length_top_left}" n_bars="${n_bars_top}" slope="${body_top_slope}" mirror="-1" />
+    <xacro:bar_in_row note="Fs4" parent="body_top" id="3" left_x="${top_left_center_x}" left_y="${top_left_center_y}" left_z="${top_left_center_z}" length_diff="${body_top_length_diff}" bar_length_left="${bar_length_top_left}" n_bars="${n_bars_top}" slope="${body_top_slope}" mirror="-1" />
+    <xacro:bar_in_row note="Gs4" parent="body_top" id="4" left_x="${top_left_center_x}" left_y="${top_left_center_y}" left_z="${top_left_center_z}" length_diff="${body_top_length_diff}" bar_length_left="${bar_length_top_left}" n_bars="${n_bars_top}" slope="${body_top_slope}" mirror="-1" />
+    <xacro:bar_in_row note="As4" parent="body_top" id="5" left_x="${top_left_center_x}" left_y="${top_left_center_y}" left_z="${top_left_center_z}" length_diff="${body_top_length_diff}" bar_length_left="${bar_length_top_left}" n_bars="${n_bars_top}" slope="${body_top_slope}" mirror="-1" />
     <!-- <xacro:bar_in_row note="" parent="body_top" id="6" left_x="${top_left_center_x}" left_y="${top_left_center_y}" left_z="${top_left_center_z}" length_diff="${body_top_length_diff}" bar_length_left="${bar_length_top_left}" n_bars="${n_bars_top}" slope="${body_top_slope}" mirror="-1" /> -->
-    <xacro:bar_in_row note="C#5" parent="body_top" id="7" left_x="${top_left_center_x}" left_y="${top_left_center_y}" left_z="${top_left_center_z}" length_diff="${body_top_length_diff}" bar_length_left="${bar_length_top_left}" n_bars="${n_bars_top}" slope="${body_top_slope}" mirror="-1" />
-    <xacro:bar_in_row note="D#5" parent="body_top" id="8" left_x="${top_left_center_x}" left_y="${top_left_center_y}" left_z="${top_left_center_z}" length_diff="${body_top_length_diff}" bar_length_left="${bar_length_top_left}" n_bars="${n_bars_top}" slope="${body_top_slope}" mirror="-1" />
+    <xacro:bar_in_row note="Cs5" parent="body_top" id="7" left_x="${top_left_center_x}" left_y="${top_left_center_y}" left_z="${top_left_center_z}" length_diff="${body_top_length_diff}" bar_length_left="${bar_length_top_left}" n_bars="${n_bars_top}" slope="${body_top_slope}" mirror="-1" />
+    <xacro:bar_in_row note="Ds5" parent="body_top" id="8" left_x="${top_left_center_x}" left_y="${top_left_center_y}" left_z="${top_left_center_z}" length_diff="${body_top_length_diff}" bar_length_left="${bar_length_top_left}" n_bars="${n_bars_top}" slope="${body_top_slope}" mirror="-1" />
     <!-- <xacro:bar_in_row note="" parent="body_top" id="9" left_x="${top_left_center_x}" left_y="${top_left_center_y}" left_z="${top_left_center_z}" length_diff="${body_top_length_diff}" bar_length_left="${bar_length_top_left}" n_bars="${n_bars_top}" slope="${body_top_slope}" mirror="-1" /> -->
-    <xacro:bar_in_row note="F#5" parent="body_top" id="10" left_x="${top_left_center_x}" left_y="${top_left_center_y}" left_z="${top_left_center_z}" length_diff="${body_top_length_diff}" bar_length_left="${bar_length_top_left}" n_bars="${n_bars_top}" slope="${body_top_slope}" mirror="-1" />
-    <xacro:bar_in_row note="G#5" parent="body_top" id="11" left_x="${top_left_center_x}" left_y="${top_left_center_y}" left_z="${top_left_center_z}" length_diff="${body_top_length_diff}" bar_length_left="${bar_length_top_left}" n_bars="${n_bars_top}" slope="${body_top_slope}" mirror="-1" />
-    <xacro:bar_in_row note="A#5" parent="body_top" id="12" left_x="${top_left_center_x}" left_y="${top_left_center_y}" left_z="${top_left_center_z}" length_diff="${body_top_length_diff}" bar_length_left="${bar_length_top_left}" n_bars="${n_bars_top}" slope="${body_top_slope}" mirror="-1" />
+    <xacro:bar_in_row note="Fs5" parent="body_top" id="10" left_x="${top_left_center_x}" left_y="${top_left_center_y}" left_z="${top_left_center_z}" length_diff="${body_top_length_diff}" bar_length_left="${bar_length_top_left}" n_bars="${n_bars_top}" slope="${body_top_slope}" mirror="-1" />
+    <xacro:bar_in_row note="Gs5" parent="body_top" id="11" left_x="${top_left_center_x}" left_y="${top_left_center_y}" left_z="${top_left_center_z}" length_diff="${body_top_length_diff}" bar_length_left="${bar_length_top_left}" n_bars="${n_bars_top}" slope="${body_top_slope}" mirror="-1" />
+    <xacro:bar_in_row note="As5" parent="body_top" id="12" left_x="${top_left_center_x}" left_y="${top_left_center_y}" left_z="${top_left_center_z}" length_diff="${body_top_length_diff}" bar_length_left="${bar_length_top_left}" n_bars="${n_bars_top}" slope="${body_top_slope}" mirror="-1" />
     <!-- <xacro:bar_in_rbar_in_rowow note="" parent="body_top" id="13" left_x="${top_left_center_x}" left_y="${top_left_center_y}" left_z="${top_left_center_z}" length_diff="${body_top_length_diff}" bar_length_left="${bar_length_top_left}" n_bars="${n_bars_top}" slope="${body_top_slope}" mirror="-1" /> -->
-    <xacro:bar_in_row note="C#6" parent="body_top" id="14" left_x="${top_left_center_x}" left_y="${top_left_center_y}" left_z="${top_left_center_z}" length_diff="${body_top_length_diff}" bar_length_left="${bar_length_top_left}" n_bars="${n_bars_top}" slope="${body_top_slope}" mirror="-1" />
-    <xacro:bar_in_row note="D#6" parent="body_top" id="15" left_x="${top_left_center_x}" left_y="${top_left_center_y}" left_z="${top_left_center_z}" length_diff="${body_top_length_diff}" bar_length_left="${bar_length_top_left}" n_bars="${n_bars_top}" slope="${body_top_slope}" mirror="-1" />
+    <xacro:bar_in_row note="Cs6" parent="body_top" id="14" left_x="${top_left_center_x}" left_y="${top_left_center_y}" left_z="${top_left_center_z}" length_diff="${body_top_length_diff}" bar_length_left="${bar_length_top_left}" n_bars="${n_bars_top}" slope="${body_top_slope}" mirror="-1" />
+    <xacro:bar_in_row note="Ds6" parent="body_top" id="15" left_x="${top_left_center_x}" left_y="${top_left_center_y}" left_z="${top_left_center_z}" length_diff="${body_top_length_diff}" bar_length_left="${bar_length_top_left}" n_bars="${n_bars_top}" slope="${body_top_slope}" mirror="-1" />
     <!-- <xacro:bar_in_row note="" parent="body_top" id="16" left_x="${top_left_center_x}" left_y="${top_left_center_y}" left_z="${top_left_center_z}" length_diff="${body_top_length_diff}" bar_length_left="${bar_length_top_left}" n_bars="${n_bars_top}" slope="${body_top_slope}" mirror="-1" /> -->
-    <xacro:bar_in_row note="F#6" parent="body_top" id="17" left_x="${top_left_center_x}" left_y="${top_left_center_y}" left_z="${top_left_center_z}" length_diff="${body_top_length_diff}" bar_length_left="${bar_length_top_left}" n_bars="${n_bars_top}" slope="${body_top_slope}" mirror="-1" />
-    <xacro:bar_in_row note="G#6" parent="body_top" id="18" left_x="${top_left_center_x}" left_y="${top_left_center_y}" left_z="${top_left_center_z}" length_diff="${body_top_length_diff}" bar_length_left="${bar_length_top_left}" n_bars="${n_bars_top}" slope="${body_top_slope}" mirror="-1" />
-    <xacro:bar_in_row note="A#6" parent="body_top" id="19" left_x="${top_left_center_x}" left_y="${top_left_center_y}" left_z="${top_left_center_z}" length_diff="${body_top_length_diff}" bar_length_left="${bar_length_top_left}" n_bars="${n_bars_top}" slope="${body_top_slope}" mirror="-1" />
+    <xacro:bar_in_row note="Fs6" parent="body_top" id="17" left_x="${top_left_center_x}" left_y="${top_left_center_y}" left_z="${top_left_center_z}" length_diff="${body_top_length_diff}" bar_length_left="${bar_length_top_left}" n_bars="${n_bars_top}" slope="${body_top_slope}" mirror="-1" />
+    <xacro:bar_in_row note="Gs6" parent="body_top" id="18" left_x="${top_left_center_x}" left_y="${top_left_center_y}" left_z="${top_left_center_z}" length_diff="${body_top_length_diff}" bar_length_left="${bar_length_top_left}" n_bars="${n_bars_top}" slope="${body_top_slope}" mirror="-1" />
+    <xacro:bar_in_row note="As6" parent="body_top" id="19" left_x="${top_left_center_x}" left_y="${top_left_center_y}" left_z="${top_left_center_z}" length_diff="${body_top_length_diff}" bar_length_left="${bar_length_top_left}" n_bars="${n_bars_top}" slope="${body_top_slope}" mirror="-1" />
 </xacro:macro>
 <xacro:marimba name="marimba" />

File: marimbabot_description/urdf/marimbabot_ur5.urdf.xacro (robot description, xacro)
@@ -10,4 +10,5 @@
   <xacro:include filename="$(find tams_ur5_description)/urdf/arm.urdf.xacro" />
   <xacro:include filename="$(find marimbabot_description)/urdf/marimba.urdf.xacro" />
+  <xacro:include filename="$(find marimbabot_description)/urdf/gazebo_gripper_transmissions.xacro" />
   <link name="world" />
   <joint name="world_floor_joint" type="fixed">

File: marimbabot_description/urdf/utilities.xacro (robot description, xacro)
@@ -41,4 +41,5 @@
   <child link="${child}"/>
   <xacro:insert_block name="origin" />
+  <limit effort="30" velocity="1.0" lower="-0.001" upper="0.001" />
 </joint>
 </xacro:macro>
