Commit message: Gazebo simulation (#80)
* Change the bar names # -> s

* WIP: Gazebo simulation

* WIP gazebo

* add tams_ur5_gazebo to workspace

* remove redundant gazebo control plugin

* conditional loading for mallet

* split controllers into separate YAML files

* revert backed up files

* split controllers

* revert commented moveit controllers

* update inertia parameters

* fine tune PID parameters

* change # to s in bar frame names

* slightly more optimal pid params

* remove unused args and add doc

* remove comments

* remove confusing unused file

* remove comments

---------

Co-authored-by: TAMS Project 2022 <tams@informatik.uni-hamburg.de>
Co-authored-by: berkgungor <brekgungor@gmail.com>

File: marimbabot_description/urdf/marimba.urdf.xacro (robot description, xacro)
@@ -10,4 +10,5 @@
     z: points towards the ceiling, according to right hand rule
 Changelog:
+    2023.04.20 TODO
     2023.03.02 Named and correctly positioned bar frames
                Added side boxes
@@ -15,6 +16,4 @@
     2023.01.19 Row of keys working
     2023.01.04 First version created
-TODO:
-    - prismatic joints instead of fixed ones for the bars
 -->
 <!-- Number of bars (including "missing" ones in the top row) -->
@@ -112,7 +111,16 @@
     </collision>
     </link>
-    <xacro:tams_fixedjoint name="bar_${note}/fixedjoint" parent="${parent}" child="bar_${note}" >
+    <xacro:tams_z_joint name="bar_${note}/joint" parent="${parent}" child="bar_${note}" >
         <origin xyz="${pos}" rpy="0 0 0" />
-    </xacro:tams_fixedjoint>
+    </xacro:tams_z_joint>
+    <transmission name="bar_${note}/joint_transmission">
+        <type>transmission_interface/SimpleTransmission</type>
+        <joint name="bar_${note}/joint">
+        <hardwareInterface>hardware_interface/EffortJointInterface</hardwareInterface>
+        </joint>
+        <actuator name="bar_${note}/joint_motor">
+        <mechanicalReduction>1</mechanicalReduction>
+        </actuator>
+    </transmission>
 </xacro:macro>
 <!-- Wrapper for a row of bars, computes the position and length based on fixed measurements -->
@@ -140,16 +148,4 @@
         <kp>1000000.0</kp>
         <kd>1.0</kd>
-    </gazebo>
-    <gazebo>
-        <plugin filename="libgazebo_ros_control.so" name="${name}_gazebo_ros_control">
-            <!-- don't add the robotNamespace here unless you really want it -->
-            <!-- <robotNamespace>${name}/</robotNamespace> -->
-            <!-- <robotNamespace>/</robotNamespaside_left_posce> -->
-            <robotParam>robot_description</robotParam>
-            <robotSimType>gazebo_ros_control/DefaultRobotHWSim</robotSimType>
-            <legacyModeNS>true</legacyModeNS>
-            <!-- specify control period, default is to use the physics period -->
-            <!-- <controlPeriod>0.0333</controlPeriod> -->
-        </plugin>
     </gazebo>
     <!-- Bottom body -->
@@ -319,24 +315,24 @@
     <!-- Top row of bars -->
     <xacro:property name="body_top_length_diff" value="${bar_length_top_right - bar_length_top_left}" />
-    <xacro:bar_in_row note="C#4" parent="body_top" id="0" left_x="${top_left_center_x}" left_y="${top_left_center_y}" left_z="${top_left_center_z}" length_diff="${body_top_length_diff}" bar_length_left="${bar_length_top_left}" n_bars="${n_bars_top}" slope="${body_top_slope}" mirror="-1" />
-    <xacro:bar_in_row note="D#4" parent="body_top" id="1" left_x="${top_left_center_x}" left_y="${top_left_center_y}" left_z="${top_left_center_z}" length_diff="${body_top_length_diff}" bar_length_left="${bar_length_top_left}" n_bars="${n_bars_top}" slope="${body_top_slope}" mirror="-1" />
+    <xacro:bar_in_row note="Cs4" parent="body_top" id="0" left_x="${top_left_center_x}" left_y="${top_left_center_y}" left_z="${top_left_center_z}" length_diff="${body_top_length_diff}" bar_length_left="${bar_length_top_left}" n_bars="${n_bars_top}" slope="${body_top_slope}" mirror="-1" />
+    <xacro:bar_in_row note="Ds4" parent="body_top" id="1" left_x="${top_left_center_x}" left_y="${top_left_center_y}" left_z="${top_left_center_z}" length_diff="${body_top_length_diff}" bar_length_left="${bar_length_top_left}" n_bars="${n_bars_top}" slope="${body_top_slope}" mirror="-1" />
     <!-- <xacro:bar_in_row note="" parent="body_top" id="2" left_x="${top_left_center_x}" left_y="${top_left_center_y}" left_z="${top_left_center_z}" length_diff="${body_top_length_diff}" bar_length_left="${bar_length_top_left}" n_bars="${n_bars_top}" slope="${body_top_slope}" mirror="-1" /> -->
-    <xacro:bar_in_row note="F#4" parent="body_top" id="3" left_x="${top_left_center_x}" left_y="${top_left_center_y}" left_z="${top_left_center_z}" length_diff="${body_top_length_diff}" bar_length_left="${bar_length_top_left}" n_bars="${n_bars_top}" slope="${body_top_slope}" mirror="-1" />
-    <xacro:bar_in_row note="G#4" parent="body_top" id="4" left_x="${top_left_center_x}" left_y="${top_left_center_y}" left_z="${top_left_center_z}" length_diff="${body_top_length_diff}" bar_length_left="${bar_length_top_left}" n_bars="${n_bars_top}" slope="${body_top_slope}" mirror="-1" />
-    <xacro:bar_in_row note="A#4" parent="body_top" id="5" left_x="${top_left_center_x}" left_y="${top_left_center_y}" left_z="${top_left_center_z}" length_diff="${body_top_length_diff}" bar_length_left="${bar_length_top_left}" n_bars="${n_bars_top}" slope="${body_top_slope}" mirror="-1" />
+    <xacro:bar_in_row note="Fs4" parent="body_top" id="3" left_x="${top_left_center_x}" left_y="${top_left_center_y}" left_z="${top_left_center_z}" length_diff="${body_top_length_diff}" bar_length_left="${bar_length_top_left}" n_bars="${n_bars_top}" slope="${body_top_slope}" mirror="-1" />
+    <xacro:bar_in_row note="Gs4" parent="body_top" id="4" left_x="${top_left_center_x}" left_y="${top_left_center_y}" left_z="${top_left_center_z}" length_diff="${body_top_length_diff}" bar_length_left="${bar_length_top_left}" n_bars="${n_bars_top}" slope="${body_top_slope}" mirror="-1" />
+    <xacro:bar_in_row note="As4" parent="body_top" id="5" left_x="${top_left_center_x}" left_y="${top_left_center_y}" left_z="${top_left_center_z}" length_diff="${body_top_length_diff}" bar_length_left="${bar_length_top_left}" n_bars="${n_bars_top}" slope="${body_top_slope}" mirror="-1" />
     <!-- <xacro:bar_in_row note="" parent="body_top" id="6" left_x="${top_left_center_x}" left_y="${top_left_center_y}" left_z="${top_left_center_z}" length_diff="${body_top_length_diff}" bar_length_left="${bar_length_top_left}" n_bars="${n_bars_top}" slope="${body_top_slope}" mirror="-1" /> -->
-    <xacro:bar_in_row note="C#5" parent="body_top" id="7" left_x="${top_left_center_x}" left_y="${top_left_center_y}" left_z="${top_left_center_z}" length_diff="${body_top_length_diff}" bar_length_left="${bar_length_top_left}" n_bars="${n_bars_top}" slope="${body_top_slope}" mirror="-1" />
-    <xacro:bar_in_row note="D#5" parent="body_top" id="8" left_x="${top_left_center_x}" left_y="${top_left_center_y}" left_z="${top_left_center_z}" length_diff="${body_top_length_diff}" bar_length_left="${bar_length_top_left}" n_bars="${n_bars_top}" slope="${body_top_slope}" mirror="-1" />
+    <xacro:bar_in_row note="Cs5" parent="body_top" id="7" left_x="${top_left_center_x}" left_y="${top_left_center_y}" left_z="${top_left_center_z}" length_diff="${body_top_length_diff}" bar_length_left="${bar_length_top_left}" n_bars="${n_bars_top}" slope="${body_top_slope}" mirror="-1" />
+    <xacro:bar_in_row note="Ds5" parent="body_top" id="8" left_x="${top_left_center_x}" left_y="${top_left_center_y}" left_z="${top_left_center_z}" length_diff="${body_top_length_diff}" bar_length_left="${bar_length_top_left}" n_bars="${n_bars_top}" slope="${body_top_slope}" mirror="-1" />
     <!-- <xacro:bar_in_row note="" parent="body_top" id="9" left_x="${top_left_center_x}" left_y="${top_left_center_y}" left_z="${top_left_center_z}" length_diff="${body_top_length_diff}" bar_length_left="${bar_length_top_left}" n_bars="${n_bars_top}" slope="${body_top_slope}" mirror="-1" /> -->
-    <xacro:bar_in_row note="F#5" parent="body_top" id="10" left_x="${top_left_center_x}" left_y="${top_left_center_y}" left_z="${top_left_center_z}" length_diff="${body_top_length_diff}" bar_length_left="${bar_length_top_left}" n_bars="${n_bars_top}" slope="${body_top_slope}" mirror="-1" />
-    <xacro:bar_in_row note="G#5" parent="body_top" id="11" left_x="${top_left_center_x}" left_y="${top_left_center_y}" left_z="${top_left_center_z}" length_diff="${body_top_length_diff}" bar_length_left="${bar_length_top_left}" n_bars="${n_bars_top}" slope="${body_top_slope}" mirror="-1" />
-    <xacro:bar_in_row note="A#5" parent="body_top" id="12" left_x="${top_left_center_x}" left_y="${top_left_center_y}" left_z="${top_left_center_z}" length_diff="${body_top_length_diff}" bar_length_left="${bar_length_top_left}" n_bars="${n_bars_top}" slope="${body_top_slope}" mirror="-1" />
+    <xacro:bar_in_row note="Fs5" parent="body_top" id="10" left_x="${top_left_center_x}" left_y="${top_left_center_y}" left_z="${top_left_center_z}" length_diff="${body_top_length_diff}" bar_length_left="${bar_length_top_left}" n_bars="${n_bars_top}" slope="${body_top_slope}" mirror="-1" />
+    <xacro:bar_in_row note="Gs5" parent="body_top" id="11" left_x="${top_left_center_x}" left_y="${top_left_center_y}" left_z="${top_left_center_z}" length_diff="${body_top_length_diff}" bar_length_left="${bar_length_top_left}" n_bars="${n_bars_top}" slope="${body_top_slope}" mirror="-1" />
+    <xacro:bar_in_row note="As5" parent="body_top" id="12" left_x="${top_left_center_x}" left_y="${top_left_center_y}" left_z="${top_left_center_z}" length_diff="${body_top_length_diff}" bar_length_left="${bar_length_top_left}" n_bars="${n_bars_top}" slope="${body_top_slope}" mirror="-1" />
     <!-- <xacro:bar_in_rbar_in_rowow note="" parent="body_top" id="13" left_x="${top_left_center_x}" left_y="${top_left_center_y}" left_z="${top_left_center_z}" length_diff="${body_top_length_diff}" bar_length_left="${bar_length_top_left}" n_bars="${n_bars_top}" slope="${body_top_slope}" mirror="-1" /> -->
-    <xacro:bar_in_row note="C#6" parent="body_top" id="14" left_x="${top_left_center_x}" left_y="${top_left_center_y}" left_z="${top_left_center_z}" length_diff="${body_top_length_diff}" bar_length_left="${bar_length_top_left}" n_bars="${n_bars_top}" slope="${body_top_slope}" mirror="-1" />
-    <xacro:bar_in_row note="D#6" parent="body_top" id="15" left_x="${top_left_center_x}" left_y="${top_left_center_y}" left_z="${top_left_center_z}" length_diff="${body_top_length_diff}" bar_length_left="${bar_length_top_left}" n_bars="${n_bars_top}" slope="${body_top_slope}" mirror="-1" />
+    <xacro:bar_in_row note="Cs6" parent="body_top" id="14" left_x="${top_left_center_x}" left_y="${top_left_center_y}" left_z="${top_left_center_z}" length_diff="${body_top_length_diff}" bar_length_left="${bar_length_top_left}" n_bars="${n_bars_top}" slope="${body_top_slope}" mirror="-1" />
+    <xacro:bar_in_row note="Ds6" parent="body_top" id="15" left_x="${top_left_center_x}" left_y="${top_left_center_y}" left_z="${top_left_center_z}" length_diff="${body_top_length_diff}" bar_length_left="${bar_length_top_left}" n_bars="${n_bars_top}" slope="${body_top_slope}" mirror="-1" />
     <!-- <xacro:bar_in_row note="" parent="body_top" id="16" left_x="${top_left_center_x}" left_y="${top_left_center_y}" left_z="${top_left_center_z}" length_diff="${body_top_length_diff}" bar_length_left="${bar_length_top_left}" n_bars="${n_bars_top}" slope="${body_top_slope}" mirror="-1" /> -->
-    <xacro:bar_in_row note="F#6" parent="body_top" id="17" left_x="${top_left_center_x}" left_y="${top_left_center_y}" left_z="${top_left_center_z}" length_diff="${body_top_length_diff}" bar_length_left="${bar_length_top_left}" n_bars="${n_bars_top}" slope="${body_top_slope}" mirror="-1" />
-    <xacro:bar_in_row note="G#6" parent="body_top" id="18" left_x="${top_left_center_x}" left_y="${top_left_center_y}" left_z="${top_left_center_z}" length_diff="${body_top_length_diff}" bar_length_left="${bar_length_top_left}" n_bars="${n_bars_top}" slope="${body_top_slope}" mirror="-1" />
-    <xacro:bar_in_row note="A#6" parent="body_top" id="19" left_x="${top_left_center_x}" left_y="${top_left_center_y}" left_z="${top_left_center_z}" length_diff="${body_top_length_diff}" bar_length_left="${bar_length_top_left}" n_bars="${n_bars_top}" slope="${body_top_slope}" mirror="-1" />
+    <xacro:bar_in_row note="Fs6" parent="body_top" id="17" left_x="${top_left_center_x}" left_y="${top_left_center_y}" left_z="${top_left_center_z}" length_diff="${body_top_length_diff}" bar_length_left="${bar_length_top_left}" n_bars="${n_bars_top}" slope="${body_top_slope}" mirror="-1" />
+    <xacro:bar_in_row note="Gs6" parent="body_top" id="18" left_x="${top_left_center_x}" left_y="${top_left_center_y}" left_z="${top_left_center_z}" length_diff="${body_top_length_diff}" bar_length_left="${bar_length_top_left}" n_bars="${n_bars_top}" slope="${body_top_slope}" mirror="-1" />
+    <xacro:bar_in_row note="As6" parent="body_top" id="19" left_x="${top_left_center_x}" left_y="${top_left_center_y}" left_z="${top_left_center_z}" length_diff="${body_top_length_diff}" bar_length_left="${bar_length_top_left}" n_bars="${n_bars_top}" slope="${body_top_slope}" mirror="-1" />
 </xacro:macro>
 <xacro:marimba name="marimba" />

File: marimbabot_description/urdf/marimbabot_ur5.urdf.xacro (robot description, xacro)
@@ -2,13 +2,84 @@
 <robot xmlns:xacro="http://www.ros.org/wiki/xacro"
        name="marimbabot_ur5" >
+  <xacro:arg name="include_mallet" default="true" />
   <!-- tams corner -->
   <xacro:include filename="$(find tams_ur5_setup_description)/urdf/tams_corner.urdf.xacro">
-  <!-- <xacro:arg name="floating_table" value="$(arg floating_table)" />-->
-  <!-- the above argument is ignored by xacro! if you want to use this argument, try another way -->
   </xacro:include>
-  <!-- arm -->
-  <xacro:include filename="$(find tams_ur5_description)/urdf/arm.urdf.xacro" />
+  <!-- arm plus additions one by one -->  <!-- include macro definitions -->
+  <xacro:include filename="$(find tams_ur5_gazebo)/urdf/ur5_for_gazebo.urdf.xacro" />
+  <xacro:include filename="$(find robotiq_3f_gripper_visualization)/cfg/robotiq-3f-gripper_articulated_macro.xacro"/>
+  <xacro:include filename="$(find robotiq_ft_sensor)/urdf/robotiq_fts150.urdf.xacro" />
+  <xacro:include filename="$(find tams_ur5_description)/urdf/ft_adapter.urdf.xacro" />
+  <xacro:include filename="$(find tams_ur5_description)/urdf/s_model_adapter.urdf.xacro" />
+  <xacro:include filename="$(find tams_ur5_description)/urdf/plug_collision_model.urdf.xacro" />
   <xacro:include filename="$(find marimbabot_description)/urdf/marimba.urdf.xacro" />
-  <xacro:include filename="$(find marimbabot_description)/urdf/static_mallet_holder.urdf" />
+  <xacro:ur5_robot prefix="ur5_" joint_limited="false" xamla_cap="true" />
+  <!-- ft_adapter -->
+  <xacro:ft_adapter name="ft_adapter" parent="ur5_ee_link">
+    <origin xyz="0.0045 0.0 0.0" rpy="0.0 ${pi/2} 0.0" />
+  </xacro:ft_adapter>
+  <!-- ft150 -->
+  <xacro:robotiq_fts150 prefix="ft_" parent="ur5_ee_link">
+    <origin xyz="0.009 0.0 0.0" rpy="0.0 ${-pi/2} ${pi}" />
+  </xacro:robotiq_fts150>
+  <!-- tool0 frame -->
+  <link name="tool0" />
+  <joint name="ft_fts_toolside_tool0" type="fixed">
+    <parent link="ft_fts_toolside"/>
+    <child link="tool0"/>
+    <origin xyz="0.0 0.0 0.0205" rpy="0.0 ${-pi/2} 0.0"/>
+  </joint>
+  <!-- s_model_adapter -->
+  <xacro:s_model_adapter name="s_model_adapter" parent="ft_fts_toolside">
+    <origin xyz="0.0 0.0 0.015" rpy="0.0 0.0 0.0" />
+  </xacro:s_model_adapter>
+  <!-- the adaptive gripper -->
+  <xacro:robotiq-3f-gripper_articulated prefix="s_model_"/>
+  <joint name="gripper_joint" type="fixed">
+    <parent link="tool0" />
+    <child link = "s_model_palm" />
+    <origin xyz="0.057 0.0 0.0" rpy="0.0 ${pi} ${-pi/2}" />
+  </joint>
+  <!-- plug collision model -->
+  <xacro:plug_collision_model name="plug_collision_model" parent="ur5_ee_link" >
+    <origin xyz="0.0 0.0 0.0" rpy="0.0 0.0 0.0" />
+  </xacro:plug_collision_model>
+  <!-- we want Gazebo to publish joint_states for all configured joints -->
+  <gazebo>
+    <plugin filename="libgazebo_ros_control.so" name="tams_ur5_gazebo_ros_control">
+      <robotNamespace>/</robotNamespace>
+      <robotSimType>gazebo_ros_control/DefaultRobotHWSim</robotSimType>
+      <legacyModeNS>true</legacyModeNS>
+      <updateRate>100.0</updateRate>
+    </plugin>
+  </gazebo>
+  <xacro:macro name="fake_transmission" params="joint_name" >
+    <transmission name="${joint_name}_transmission">
+      <type>transmission_interface/SimpleTransmission</type>
+      <actuator name="${joint_name}_motor">
+        <mechanicalReduction>1.0</mechanicalReduction>
+      </actuator>
+      <joint name="${joint_name}">
+        <hardwareInterface>hardware_interface/EffortJointInterface</hardwareInterface>
+      </joint>
+    </transmission>
+  </xacro:macro>
+  <xacro:fake_transmission joint_name="ur5_shoulder_pan_joint" />
+  <xacro:fake_transmission joint_name="ur5_shoulder_lift_joint" />
+  <xacro:fake_transmission joint_name="ur5_elbow_joint" />
+  <xacro:fake_transmission joint_name="ur5_wrist_1_joint" />
+  <xacro:fake_transmission joint_name="ur5_wrist_2_joint" />
+  <xacro:fake_transmission joint_name="ur5_wrist_3_joint" />
+  <xacro:fake_transmission joint_name="s_model_palm_finger_1_joint" />
+  <xacro:fake_transmission joint_name="s_model_finger_1_joint_1" />
+  <xacro:fake_transmission joint_name="s_model_finger_1_joint_2" />
+  <xacro:fake_transmission joint_name="s_model_finger_1_joint_3" />
+  <xacro:fake_transmission joint_name="s_model_palm_finger_2_joint" />
+  <xacro:fake_transmission joint_name="s_model_finger_2_joint_1" />
+  <xacro:fake_transmission joint_name="s_model_finger_2_joint_2" />
+  <xacro:fake_transmission joint_name="s_model_finger_2_joint_3" />
+  <xacro:fake_transmission joint_name="s_model_finger_middle_joint_1" />
+  <xacro:fake_transmission joint_name="s_model_finger_middle_joint_2" />
+  <xacro:fake_transmission joint_name="s_model_finger_middle_joint_3" />
   <link name="world" />
   <joint name="world_floor_joint" type="fixed">
@@ -33,8 +104,11 @@
     <origin xyz="1.25 0.8 0.9" rpy="0.0 0.0 ${pi}" />
   </joint>
-  <joint name="end_mallet" type="fixed">
-    <parent link="s_model_palm" />
-    <child link = "mallet_base_link" />
-    <origin xyz="0.0 0.0 0.0" rpy="${-pi/2} 0.0 0.0" />
-  </joint>
+  <xacro:if value="$(arg include_mallet)">
+    <xacro:include filename="$(find marimbabot_description)/urdf/static_mallet_holder.urdf" />
+    <joint name="end_mallet" type="fixed">
+      <parent link="s_model_palm" />
+      <child link = "mallet_base_link" />
+      <origin xyz="0.0 0.0 0.0" rpy="${-pi/2} 0.0 0.0" />
+    </joint>
+  </xacro:if>
 </robot>

File: marimbabot_description/urdf/static_mallet_holder.urdf (robot description, URDF)
Before this commit: robot static_mallet_holder, 3 links, 2 joints
Links:
- removed link mallet_head
- added link mallet_top, mass 0.01; collision sphere radius=0.018375; visual sphere radius=0.018375
- link mallet_base_link: mass None -> 0.005
- link mallet_neck: mass None -> 0.001; geometry collision cylinder length=0.375 radius=0.0042; visual cylinder length=0.375 radius=0.0042

Commit message: add arg to use fixed joints for bars

File: marimbabot_description/urdf/marimba.urdf.xacro (robot description, xacro)
@@ -1,4 +1,5 @@
 <?xml version="1.0" ?>
 <robot name="marimba" xmlns:xacro="http://www.ros.org/wiki/xacro">
+<xacro:arg name="bars_fixed_joint" default="false" />
 <xacro:include filename="$(find marimbabot_description)/urdf/utilities.xacro" />
 <xacro:include filename="$(find marimbabot_description)/urdf/materials.xacro" />
@@ -10,5 +11,4 @@
     z: points towards the ceiling, according to right hand rule
 Changelog:
-    2023.04.20 TODO
     2023.03.02 Named and correctly positioned bar frames
                Added side boxes
@@ -75,5 +75,5 @@
     ${top_left_center_y - side_offset}
     ${bottom_left_center_z}"
-/>re
+/>
 <xacro:property name="side_right_pos" value="
     ${float(side_left_pos.split()[0])}
@@ -111,7 +111,14 @@
     </collision>
     </link>
-    <xacro:tams_z_joint name="bar_${note}/joint" parent="${parent}" child="bar_${note}" >
-        <origin xyz="${pos}" rpy="0 0 0" />
-    </xacro:tams_z_joint>
+    <xacro:if value="$(arg bars_fixed_joint)">
+        <xacro:tams_fixedjoint name="bar_${note}/joint" parent="${parent}" child="bar_${note}" >
+            <origin xyz="${pos}" rpy="0 0 0" />
+        </xacro:tams_fixedjoint>
+    </xacro:if>
+    <xacro:unless value="$(arg bars_fixed_joint)">
+        <xacro:tams_z_joint name="bar_${note}/joint" parent="${parent}" child="bar_${note}" >
+            <origin xyz="${pos}" rpy="0 0 0" />
+        </xacro:tams_z_joint>
+    </xacro:unless>
     <transmission name="bar_${note}/joint_transmission">
         <type>transmission_interface/SimpleTransmission</type>

Commit message: set side with to 0.028

File: marimbabot_description/urdf/marimba.urdf.xacro (robot description, xacro)
@@ -66,5 +66,5 @@
 <xacro:property name="top_left_center_z" value="${float(body_top_pos.split()[2]) + body_top_height / 2 + bar_height}" />
 <!-- Side boxes (left being the longer side) -->
-<xacro:property name="side_width" value="0.05" />
+<xacro:property name="side_width" value="0.028" />
 <xacro:property name="side_length_left" value="0.61" />
 <xacro:property name="side_length_right" value="0.32" />

Commit message: reduce side height

File: marimbabot_description/urdf/marimba.urdf.xacro (robot description, xacro)
@@ -70,5 +70,7 @@
 <xacro:property name="side_length_left" value="0.61" />
 <xacro:property name="side_length_right" value="0.32" />
-<xacro:property name="side_height" value="0.1" />
+<xacro:property name="side_height" value="0.07" /> <!-- 0.07 on the high side, 0.041 on the low side.
+                                                        The low side starts at 0.28 when counting from the high side.
+                                                        This is not taken into account here. -->
 <xacro:property name="side_offset" value="0.058" />
 <xacro:property name="side_left_pos" value="
