Commit message: Finalized compliant two mallet urdf model

File: marimbabot_description/urdf/two_mallet_compliance_holder.urdf.xacro (robot description, xacro)
@@ -3,5 +3,5 @@
     <link name="mallet_base_link">
         <visual>
-            <origin xyz="0.0 0.0 0.0" rpy="0.0 0.0 0.0"/>
+            <origin xyz="0.0 0.0 0.0" rpy="${-pi / 2} 0.0 0.0"/>
             <geometry>
                 <mesh filename="package://marimbabot_description/mesh/two_mallet_compliance_holder_static_element.stl" scale="0.001 0.001 0.001"/>
@@ -12,7 +12,7 @@
         </visual>
         <collision>
-            <origin xyz="0.0 0.0 0.0" rpy="0.0 0.0 0.0"/>
+            <origin xyz="0.0 0.0 ${0.06/2}" rpy="0.0 0.0 0.0"/>
             <geometry>
-                <box size="0.08 0.06 0.070"/>
+                <box size="0.08 0.07 0.06"/>
             </geometry>
         </collision>
@@ -20,15 +20,18 @@
     <link name="mallet_servo_box">
         <visual>
-            <origin xyz="0.0 0.0 0.0" rpy="0.0 0.0 0.0"/>
+            <origin xyz="0.0 0.0 0.0" rpy="${-pi / 2} 0.0 0.0"/>
             <geometry>
                 <mesh filename="package://marimbabot_description/mesh/two_mallet_compliance_holder_dynamic_element.stl" scale="0.001 0.001 0.001"/>
             </geometry>
+            <material name="mallet_holder_white">
+                <color rgba="1.0 1.0 1.0 1.0"/>
+            </material>
         </visual>
     </link>
     <link name="mallet_base_box_1">
         <collision>
-            <origin xyz="0.0 0.0 0.45" rpy="0.0 0.0 0.0"/>
+            <origin xyz="0.0 0.0 0.045" rpy="0.0 0.0 0.0"/>
             <geometry>
-                <box size="0.033 0.033 0.09"/>
+                <box size="0.033 0.09 0.09"/>
             </geometry>
         </collision>
@@ -36,7 +39,7 @@
     <link name="mallet_base_box_2">
         <collision>
-            <origin xyz="0.0 0.0 0.0" rpy="0.0 0.0 0.0"/>
+            <origin xyz="0.0 0.0 0.045" rpy="0.0 0.0 0.0"/>
             <geometry>
-                <box size="0.033 0.033 0.09"/>
+                <box size="0.033 0.09 0.09"/>
             </geometry>
         </collision>
@@ -44,5 +47,5 @@
     <link name="mallet_neck_1">
         <collision>
-            <origin xyz="0.0 0.0 0.1825" rpy="0.0 0.0 0.0"/>
+            <origin xyz="0.0 0.0 ${0.1825+0.005}" rpy="0.0 0.0 0.0"/>
             <geometry>
                 <cylinder radius="0.0042" length="0.375"/>
@@ -52,5 +55,5 @@
     <link name="mallet_neck_2">
         <collision>
-            <origin xyz="0.0 0.0 0.1825" rpy="0.0 0.0 0.0"/>
+            <origin xyz="0.0 0.0 ${0.1825+0.005}" rpy="0.0 0.0 0.0"/>
             <geometry>
                 <cylinder radius="0.0042" length="0.375"/>
@@ -60,6 +63,5 @@
     <link name="mallet_top_1">
         <collision>
-            <origin xyz="0.0 0.0 0.013625" rpy="0.0 0.0 0.0"/>
-            <!-- 0.018375 -->
+            <origin xyz="0.0 0.0 0.0" rpy="0.0 0.0 0.0"/>
             <geometry>
                 <sphere radius="0.018375"/>
@@ -69,6 +71,5 @@
     <link name="mallet_top_2">
         <collision>
-            <origin xyz="0.0 0.0 0.013625" rpy="0.0 0.0 0.0"/>
-            <!-- 0.018375 -->
+            <origin xyz="0.0 0.0 0.0" rpy="0.0 0.0 0.0"/>
             <geometry>
                 <sphere radius="0.018375"/>
@@ -79,36 +80,37 @@
         <parent link="mallet_base_link"/>
         <child link="mallet_base_box_1"/>
-        <origin xyz="0.0 0.0 0.45"/>
+        <origin xyz="0.0225 0.003 0.072"/>
     </joint>
     <joint name="mallet_finger" type="revolute">
         <parent link="mallet_base_link"/>
         <child link="mallet_servo_box"/>
-        <origin xyz="0.0 0.0 0.0"/>
-        <limit lower="0.0" upper="1.602" effort="1.0" velocity="7.0"/>
+        <origin xyz="-0.02 0.0 0.0368"/>
+        <limit lower="0.0" upper="0.801" effort="1.0" velocity="7.0"/>
+        <axis xyz="0.0 -1.0 0.0"/>
     </joint>
     <joint name="mallet_group_1_start_link" type="fixed">
         <parent link="mallet_base_box_1"/>
         <child link="mallet_neck_1"/>
-        <origin xyz="0.0 0.0 0.0292"/>
+        <origin xyz="0.0 0.0 0.015"/>
     </joint>
     <joint name="mallet_group_1_2nd_link" type="fixed">
         <parent link="mallet_neck_1"/>
         <child link="mallet_top_1"/>
-        <origin xyz="0.0 0.0 0.365"/>
+        <origin xyz="0.0 0.0 ${0.365+0.018375}"/>
     </joint>
     <joint name="mallet_group_2_start_link" type="fixed">
         <parent link="mallet_servo_box"/>
         <child link="mallet_base_box_2"/>
-        <origin xyz="0.0 0.0 0.0"/>
+        <origin xyz="0.0075 0.003 0.0353"/>
     </joint>
     <joint name="mallet_group_2_2nd_link" type="fixed">
         <parent link="mallet_base_box_2"/>
         <child link="mallet_neck_2"/>
-        <origin xyz="0.0 0.0 0.0292"/>
+        <origin xyz="0.0 0.0 0.015"/>
     </joint>
     <joint name="mallet_group_2_3rd_link" type="fixed">
         <parent link="mallet_neck_2"/>
         <child link="mallet_top_2"/>
-        <origin xyz="0.0 0.0 0.365"/>
+        <origin xyz="0.0 0.0 ${0.365+0.018375}"/>
     </joint>
 </robot>

Commit message: Changed mallet_top to mallet_head

File: marimbabot_description/urdf/two_mallet_compliance_holder.urdf.xacro (robot description, xacro)
@@ -61,5 +61,5 @@
         </collision>
     </link>
-    <link name="mallet_top_1">
+    <link name="mallet_head_1">
         <collision>
             <origin xyz="0.0 0.0 0.0" rpy="0.0 0.0 0.0"/>
@@ -69,5 +69,5 @@
         </collision>
     </link>
-    <link name="mallet_top_2">
+    <link name="mallet_head_2">
         <collision>
             <origin xyz="0.0 0.0 0.0" rpy="0.0 0.0 0.0"/>
@@ -96,5 +96,5 @@
     <joint name="mallet_group_1_2nd_link" type="fixed">
         <parent link="mallet_neck_1"/>
-        <child link="mallet_top_1"/>
+        <child link="mallet_head_1"/>
         <origin xyz="0.0 0.0 ${0.365+0.018375}"/>
     </joint>
@@ -111,5 +111,5 @@
     <joint name="mallet_group_2_3rd_link" type="fixed">
         <parent link="mallet_neck_2"/>
-        <child link="mallet_top_2"/>
+        <child link="mallet_head_2"/>
         <origin xyz="0.0 0.0 ${0.365+0.018375}"/>
     </joint>

Commit message: Changed two mallet xacro model to reflect the newest iteration of the model

File: marimbabot_description/urdf/two_mallet_compliance_holder.urdf.xacro (robot description, xacro)
@@ -3,7 +3,7 @@
     <link name="mallet_base_link">
         <visual>
-            <origin xyz="0.0 0.0 0.0" rpy="${-pi / 2} 0.0 0.0"/>
+            <origin xyz="${(7-77/2)/1000} ${(6-(68.4+6+6)/2)/1000} ${110/1000}" rpy="${-pi / 2} 0.0 0.0"/>
             <geometry>
-                <mesh filename="package://marimbabot_description/mesh/two_mallet_compliance_holder_static_element.stl" scale="0.001 0.001 0.001"/>
+                <mesh filename="package://marimbabot_description/mesh/two_mallet_base_element.stl" scale="0.001 0.001 0.001"/>
             </geometry>
             <material name="mallet_holder_white">
@@ -12,7 +12,7 @@
         </visual>
         <collision>
-            <origin xyz="0.0 0.0 ${0.06/2}" rpy="0.0 0.0 0.0"/>
+            <origin xyz="0.0 0.0 ${0.11/2}" rpy="0.0 0.0 0.0"/>
             <geometry>
-                <box size="0.08 0.07 0.06"/>
+                <box size="0.077 ${(68.4+6+6)/1000} 0.11"/>
             </geometry>
         </collision>
@@ -20,7 +20,7 @@
     <link name="mallet_servo_box">
         <visual>
-            <origin xyz="0.0 0.0 0.0" rpy="${-pi / 2} 0.0 0.0"/>
+            <origin xyz="${-(10)/1000} ${(6-(68.4+6+6)/2)/1000} ${(13.3+10)/1000}" rpy="${-pi / 2} 0.0 0.0"/>
             <geometry>
-                <mesh filename="package://marimbabot_description/mesh/two_mallet_compliance_holder_dynamic_element.stl" scale="0.001 0.001 0.001"/>
+                <mesh filename="package://marimbabot_description/mesh/two_mallet_servo_element.stl" scale="0.001 0.001 0.001"/>
             </geometry>
             <material name="mallet_holder_white">
@@ -30,4 +30,13 @@
     </link>
     <link name="mallet_base_box_1">
+        <visual>
+            <origin xyz="0.0 0.0 ${(90/2)/1000}" rpy="${-pi / 2} ${-pi / 2} 0.0"/>
+            <geometry>
+                <mesh filename="package://marimbabot_description/mesh/mallet_double_flex.stl" scale="0.001 0.001 0.001"/>
+            </geometry>
+            <material name="mallet_holder_white">
+                <color rgba="1.0 1.0 1.0 1.0"/>
+            </material>
+        </visual>
         <collision>
             <origin xyz="0.0 0.0 0.045" rpy="0.0 0.0 0.0"/>
@@ -38,4 +47,13 @@
     </link>
     <link name="mallet_base_box_2">
+        <visual>
+            <origin xyz="0.0 0.0 ${(90/2)/1000}" rpy="${-pi / 2} ${-pi / 2} ${pi}"/>
+            <geometry>
+                <mesh filename="package://marimbabot_description/mesh/mallet_double_flex.stl" scale="0.001 0.001 0.001"/>
+            </geometry>
+            <material name="mallet_holder_white">
+                <color rgba="1.0 1.0 1.0 1.0"/>
+            </material>
+        </visual>
         <collision>
             <origin xyz="0.0 0.0 0.045" rpy="0.0 0.0 0.0"/>
@@ -80,10 +98,10 @@
         <parent link="mallet_base_link"/>
         <child link="mallet_base_box_1"/>
-        <origin xyz="0.0225 0.003 0.072"/>
+        <origin xyz="${(77/2-35/2)/1000} 0.0038 ${(110+12-0.2)/1000}"/>
     </joint>
     <joint name="mallet_finger" type="revolute">
         <parent link="mallet_base_link"/>
         <child link="mallet_servo_box"/>
-        <origin xyz="-0.02 0.0 0.0368"/>
+        <origin xyz="${(-77/2+10+7)/1000} 0.0 ${0.0368+(110-60)/1000}"/>
         <limit lower="0.0" upper="0.801" effort="1.0" velocity="7.0"/>
         <axis xyz="0.0 -1.0 0.0"/>
@@ -102,5 +120,5 @@
         <parent link="mallet_servo_box"/>
         <child link="mallet_base_box_2"/>
-        <origin xyz="0.0075 0.003 0.0353"/>
+        <origin xyz="0.0075 0.0038 0.0351"/>
     </joint>
     <joint name="mallet_group_2_2nd_link" type="fixed">

Commit message: Adjusting limit in the actual urdf file

File: marimbabot_description/urdf/two_mallet_compliance_holder.urdf.xacro (robot description, xacro)
@@ -104,5 +104,5 @@
         <child link="mallet_servo_box"/>
         <origin xyz="${(-77/2+10+7)/1000} 0.0 ${0.0368+(110-60)/1000}"/>
-        <limit lower="0.0" upper="0.801" effort="1.0" velocity="7.0"/>
+        <limit lower="0.0" upper="1.22" effort="1.0" velocity="7.0"/>
         <axis xyz="0.0 -1.0 0.0"/>
     </joint>

Commit message: Added collision for battery area

File: marimbabot_description/urdf/two_mallet_compliance_holder.urdf.xacro (robot description, xacro)
@@ -15,4 +15,12 @@
             <geometry>
                 <box size="0.077 ${(68.4+6+6)/1000} 0.11"/>
+            </geometry>
+        </collision>
+    </link>
+    <link name="mallet_battery_collision">
+        <collision>
+            <origin xyz="-${0.026/2} -${0.04/2} ${0.11/2}" rpy="0.0 0.0 0.0"/>
+            <geometry>
+                <box size="0.026 0.04 0.11"/>
             </geometry>
         </collision>
@@ -95,4 +103,9 @@
         </collision>
     </link>
+    <joint name="mallet_base_link_battery" type="fixed">
+        <parent link="mallet_base_link"/>
+        <child link="mallet_battery_collision"/>
+        <origin xyz="0.0115 -0.0405 0.0"/>
+    </joint>
     <joint name="mallet_base_link_group_1" type="fixed">
         <parent link="mallet_base_link"/>

Commit message: Add collision to mallet_servo_box (was a warning)

File: marimbabot_description/urdf/two_mallet_compliance_holder.urdf.xacro (robot description, xacro)
@@ -36,4 +36,10 @@
             </material>
         </visual>
+        <collision>
+            <origin xyz="${-(10)/1000} ${(6-(68.4+6+6)/2)/1000} ${(13.3+10)/1000}" rpy="${-pi / 2} 0.0 0.0"/>
+            <geometry>
+                <mesh filename="package://marimbabot_description/mesh/two_mallet_servo_element.stl" scale="0.001 0.001 0.001"/>
+            </geometry>
+        </collision>
     </link>
     <link name="mallet_base_box_1">

Commit message: Fix 2nd mallet in Gazebo

File: marimbabot_description/urdf/two_mallet_compliance_holder.urdf.xacro (robot description, xacro)
@@ -17,4 +17,9 @@
             </geometry>
         </collision>
+        <inertial>
+            <origin xyz="0 0 0" rpy="0 0 0"/>
+            <mass value="0.01"/>
+            <inertia ixx="0.001" ixy="0" ixz="0" iyy="0.001" iyz="0" izz="0.001"/>
+        </inertial>
     </link>
     <link name="mallet_battery_collision">
@@ -42,4 +47,9 @@
             </geometry>
         </collision>
+        <inertial>
+            <origin xyz="0 0 0" rpy="0 0 0"/>
+            <mass value="0.01"/>
+            <inertia ixx="0.001" ixy="0" ixz="0" iyy="0.001" iyz="0" izz="0.001"/>
+        </inertial>
     </link>
     <link name="mallet_base_box_1">
@@ -59,4 +69,9 @@
             </geometry>
         </collision>
+        <inertial>
+            <origin xyz="0 0 0" rpy="0 0 0"/>
+            <mass value="0.01"/>
+            <inertia ixx="0.001" ixy="0" ixz="0" iyy="0.001" iyz="0" izz="0.001"/>
+        </inertial>
     </link>
     <link name="mallet_base_box_2">
@@ -76,4 +91,9 @@
             </geometry>
         </collision>
+        <inertial>
+            <origin xyz="0 0 0" rpy="0 0 0"/>
+            <mass value="0.01"/>
+            <inertia ixx="0.001" ixy="0" ixz="0" iyy="0.001" iyz="0" izz="0.001"/>
+        </inertial>
     </link>
     <link name="mallet_neck_1">
@@ -84,4 +104,9 @@
             </geometry>
         </collision>
+        <inertial>
+            <origin xyz="0 0 0" rpy="0 0 0"/>
+            <mass value="0.01"/>
+            <inertia ixx="0.001" ixy="0" ixz="0" iyy="0.001" iyz="0" izz="0.001"/>
+        </inertial>
     </link>
     <link name="mallet_neck_2">
@@ -92,4 +117,9 @@
             </geometry>
         </collision>
+        <inertial>
+            <origin xyz="0 0 0" rpy="0 0 0"/>
+            <mass value="0.01"/>
+            <inertia ixx="0.001" ixy="0" ixz="0" iyy="0.001" iyz="0" izz="0.001"/>
+        </inertial>
     </link>
     <link name="mallet_head_1">
@@ -100,4 +130,9 @@
             </geometry>
         </collision>
+        <inertial>
+            <origin xyz="0 0 0" rpy="0 0 0"/>
+            <mass value="0.01"/>
+            <inertia ixx="0.001" ixy="0" ixz="0" iyy="0.001" iyz="0" izz="0.001"/>
+        </inertial>
     </link>
     <link name="mallet_head_2">
@@ -108,4 +143,9 @@
             </geometry>
         </collision>
+        <inertial>
+            <origin xyz="0 0 0" rpy="0 0 0"/>
+            <mass value="0.01"/>
+            <inertia ixx="0.001" ixy="0" ixz="0" iyy="0.001" iyz="0" izz="0.001"/>
+        </inertial>
     </link>
     <joint name="mallet_base_link_battery" type="fixed">
@@ -126,4 +166,13 @@
         <axis xyz="0.0 -1.0 0.0"/>
     </joint>
+    <transmission name="mallet_finger_transmission">
+      <type>transmission_interface/SimpleTransmission</type>
+      <actuator name="mallet_finger_motor">
+        <mechanicalReduction>1.0</mechanicalReduction>
+      </actuator>
+      <joint name="mallet_finger">
+        <hardwareInterface>hardware_interface/EffortJointInterface</hardwareInterface>
+      </joint>
+    </transmission>
     <joint name="mallet_group_1_start_link" type="fixed">
         <parent link="mallet_base_box_1"/>

Commit message: Simulation working, add joints in the mallets for compliance

File: marimbabot_description/urdf/two_mallet_compliance_holder.urdf.xacro (robot description, xacro)
@@ -163,5 +163,5 @@
         <child link="mallet_servo_box"/>
         <origin xyz="${(-77/2+10+7)/1000} 0.0 ${0.0368+(110-60)/1000}"/>
-        <limit lower="0.0" upper="1.22" effort="1.0" velocity="7.0"/>
+        <limit lower="0.05" upper="1.22" effort="2.0" velocity="7.0"/>
         <axis xyz="0.0 -1.0 0.0"/>
     </joint>

Commit message: Remove weird collision

File: marimbabot_description/urdf/two_mallet_compliance_holder.urdf.xacro (robot description, xacro)
@@ -46,10 +46,4 @@
             </material>
         </visual>
-        <collision>
-            <origin xyz="${-(10)/1000} ${(6-(68.4+6+6)/2)/1000} ${(13.3+10)/1000}" rpy="${-pi / 2} 0.0 0.0"/>
-            <geometry>
-                <mesh filename="package://marimbabot_description/mesh/two_mallet_servo_element.stl" scale="0.001 0.001 0.001"/>
-            </geometry>
-        </collision>
         <inertial>
             <origin xyz="0 0 0" rpy="0 0 0"/>
@@ -177,5 +171,5 @@
         <child link="mallet_servo_box"/>
         <origin xyz="${(-77/2+10+7)/1000} 0.0 ${0.0368+(110-60)/1000}"/>
-        <limit lower="0.05" upper="1.22" effort="2.0" velocity="7.0"/>
+        <limit lower="0.0" upper="1.22" effort="2.0" velocity="7.0"/>
         <axis xyz="0.0 -1.0 0.0"/>
     </joint>
