Commit message: Better error handling and faster execution of command for the mallet finger (servo)

File: marimbabot_hardware/urdf/two_mallet_holder.urdf (robot description, URDF)
Before this commit: robot two_mallet_holder, 2 links, 1 joints
Joints:
- removed joint mallet_servo
- added joint mallet_finger: type revolute, parent mallet_neck, child mallet_top, origin xyz=0.0 0.0 0.0292, limit lower=0.0 upper=1.602 effort=1.0 velocity=1.0

Commit message: Getting limits from the arduino now and adjusted configuration limits for trajectories and servo speed

File: marimbabot_hardware/urdf/two_mallet_holder.urdf (robot description, URDF)
Before this commit: robot two_mallet_holder, 2 links, 1 joints
Joints:
- joint mallet_finger: limit lower=0.0 upper=1.602 effort=1.0 velocity=1.0 -> lower=0.0 upper=1.602 effort=1.0 velocity=7.0

Commit message: Adjusted hardware limits as the servo is only able to cover 180°

File: marimbabot_hardware/urdf/two_mallet_holder.urdf (robot description, URDF)
Before this commit: robot two_mallet_holder, 2 links, 1 joints
Joints:
- joint mallet_finger: limit lower=0.0 upper=1.602 effort=1.0 velocity=7.0 -> lower=0.0 upper=0.801 effort=1.0 velocity=7.0

Commit message: Adjusted hardware joint limits to be correct for the actual motion of 70°

File: marimbabot_hardware/urdf/two_mallet_holder.urdf (robot description, URDF)
Before this commit: robot two_mallet_holder, 2 links, 1 joints
Joints:
- joint mallet_finger: limit lower=0.0 upper=0.801 effort=1.0 velocity=7.0 -> lower=0.0 upper=1.22 effort=1.0 velocity=7.0
